File: USB2Serial_CH340G_v1.0.sch (EAGLE design)
At the start: 24 parts, among them CN1 UART, CN2 47346-0001, IC1 AMS1117-3.3, Q1 12MHz, U1 CH340G

Commit message: Add document number
Other:
- note added: "U2S-CH340G-0010"
Changed lines of the file:
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@@
 <text x="175.26" y="144.78" size="2.54" layer="94">UART connector and VCC selection</text>
 <text x="165.1" y="27.94" size="2.54" layer="94">(c) Andriy Golovnya</text>
+<text x="195.58" y="7.62" size="2.54" layer="94">U2S-CH340G-0010</text>
 </plain>
 <instances>
